File: keyboards/reviung41/reviung41/pcb/ver1.4/reviung41.kicad_pcb (KiCad board)
At the start: 2 copper layers, 253.3 x 107.1 mm, 111 parts, among them SW1 SW_PUSH, SW10 SW_PUSH, SW11 SW_PUSH, SW12 SW_PUSH, SW13 SW_PUSH, SW14 SW_PUSH, SW15 SW_PUSH, SW16 SW_PUSH, SW17 SW_PUSH, SW18 SW_PUSH, SW19 SW_PUSH, SW2 SW_PUSH, SW20 SW_PUSH, SW21 SW_PUSH, SW22 SW_PUSH, SW23 SW_PUSH, SW24 SW_PUSH, SW25 SW_PUSH, SW26 SW_PUSH, SW27 SW_PUSH, SW28 SW_PUSH, SW29 SW_PUSH, SW3 SW_PUSH, SW30 SW_PUSH, SW31 SW_PUSH, SW32 SW_PUSH, SW33 SW_PUSH, SW34 SW_PUSH, SW35 SW_PUSH, SW36 SW_PUSH, SW37 SW_PUSH, SW38 SW_PUSH, SW39 SW_2U_PUSH, SW4 SW_PUSH, SW40 SW_PUSH, SW41 SW_PUSH, SW5 SW_PUSH, SW6 SW_PUSH, SW7 SW_PUSH, SW8 SW_PUSH, SW9 SW_PUSH, U1 ProMicro

Commit message: add reviung41 case
Signed-off-by: Maximilian Huber <gh@maxhbr.de>
Parts:
- H1, H10, H11, H2, H3, H4, H5, H6, H7, H8, H9: footprint _reviung-kbd:HOLE -> myfootprints:HOLE
- SW1, SW10, SW11, SW12, SW13, SW14, SW15, SW16, SW17, SW18, SW19, SW2, SW20, SW21, SW22, SW23, SW24, SW25, SW26, SW27, SW28, SW29, SW3, SW30, SW31, SW32, SW33, SW34, SW35, SW36, SW37, SW38, SW4, SW40, SW41, SW5, SW6, SW7, SW8, SW9: footprint _reviung-kbd:MXOnly-1U-Hotswap -> myfootprints:MXOnly-1U-Hotswap
- SW39: footprint _reviung-kbd:MXOnly-2U-Hotswap-ReversedStabilizers -> myfootprints:MXOnly-2U-Hotswap-ReversedStabilizers
Connections:
- L11 pad 2: (no net) -> unconnected-(L11-Pad2)
- U1 pad 13: (no net) -> unconnected-(U1-Pad13)
- U1 pad 2: (no net) -> unconnected-(U1-Pad2)
- U1 pad 24: (no net) -> unconnected-(U1-Pad24)
- U1 pad 5: (no net) -> unconnected-(U1-Pad5)
- U1 pad 6: (no net) -> unconnected-(U1-Pad6)
Other:
- net class Default removed
